Commit message: simulating model on gazebo&rviz simutaneously

File: description/robot.urdf.xacro (robot description, xacro)
@@ -2,18 +2,4 @@
 <robot xmlns:xacro="http://www.ros.org/wiki/xacro"  name="robot">
   <xacro:include filename="robot_core.xacro"/>
-  <!-- <xacro:base_link/>
-  <xacro:camera_link/>
-  <xacro:lidar_link/>
-  <xacro:imu_link/>
-  <xacro:wheel_left_link/>
-  <xacro:wheel_right_link/>
-  <xacro:caster_wheel_link/>
-  <xacro:chassis_link/>
-  <xacro:camera_joint parent="base_link" child="camera_link" xyz="0.2 0 0.1" rpy="0 0 0"/>
-  <xacro:lidar_joint parent="base_link" child="lidar_link" xyz="0 0 0.1" rpy="0 0 0"/>
-  <xacro:imu_joint parent="base_link" child="imu_link" xyz="0 -0.1 0.1" rpy="0 0 0"/>
-  <xacro:wheel_left_joint parent="base_link" child="wheel_left_link" xyz="0 -0.1 -0.05" rpy="0 0 0"/>
-  <xacro:wheel_right_joint parent="base_link" child="wheel_right_link" xyz="0 0.1 -0.05" rpy="0 0 0"/>
-  <xacro:caster_wheel_joint parent="base_link" child="caster_wheel_link" xyz="-0.2 0 -0.05" rpy="0 0 0"/>
-  <xacro:chassis_joint parent="base_link" child="chassis_link" xyz="0 0 0.05" rpy="0 0 0"/> -->
+  <xacro:include filename="gazebo_control.xacro"/>
 </robot>

File: description/robot_core.xacro (robot description, xacro)
@@ -3,4 +3,18 @@
    <xacro:include filename="inertial_macros.xacro"/>
    <xacro:property name="pi" value="3.14159265359"/>
+    <xacro:property name="chassis_length" value="0.335"/>
+    <xacro:property name="chassis_width" value="0.265"/>
+    <xacro:property name="chassis_height" value="0.138"/>
+    <xacro:property name="chassis_mass" value="1.0"/>
+    <xacro:property name="wheel_radius" value="0.033"/>
+    <xacro:property name="wheel_thickness" value="0.026"/>
+    <xacro:property name="wheel_mass" value="0.05"/>
+    <xacro:property name="wheel_offset_x" value="0.226"/>
+    <xacro:property name="wheel_offset_y" value="0.1485"/>
+    <xacro:property name="wheel_offset_z" value="0.01"/>
+    <xacro:property name="caster_wheel_radius" value="0.01"/>
+    <xacro:property name="caster_wheel_mass" value="0.01"/>
+    <xacro:property name="caster_wheel_offset_x" value="0.075"/>
+    <xacro:property name="caster_wheel_offset_z" value="${wheel_offset_z - wheel_radius + caster_wheel_radius}"/>
    <material name="white">
     <color rgba="1 1 1 1" />
@@ -42,9 +56,12 @@
       </xacro:inertial_box>
    </link>
+   <gazebo reference ="chassis">
+    <material>Gazebo/Orange </material>
+   </gazebo>
    <!--LEFT WHEEL LINK-->
    <joint name="wheel_left_joint" type="continuous">
       <parent link="base_link"/>
       <child link="wheel_left"/>
-      <origin xyz="0 0.175 0" rpy="${pi/2} 0 0"/>
+      <origin xyz="0 0.175 0" rpy="-${pi/2} 0 0"/>
       <axis xyz="0 0 1"/>
    </joint>
@@ -65,4 +82,7 @@
           </xacro:inertial_cylinder>
    </link>
+   <gazebo reference ="wheel_left">
+    <material>Gazebo/Black </material>
+   </gazebo>
 <!--RIGHT WHEEL LINK-->
    <joint name="wheel_right_joint" type="continuous">
@@ -88,4 +108,7 @@
           </xacro:inertial_cylinder>
    </link>
+   <gazebo reference ="wheel_right">
+    <material>Gazebo/Black </material>
+   </gazebo>
 <!--CASTER WHEEL LINK-->
     <joint name="caster_wheel_joint" type="fixed">
@@ -99,5 +122,5 @@
                <sphere radius="0.05"/>
             </geometry>
-            <material name="yellow"/>
+            <material name="black"/>
          </visual>
           <collision>
@@ -110,3 +133,8 @@
           </xacro:inertial_sphere>
     </link>
+   <gazebo reference ="caster_wheel">
+     <material>Gazebo/Black </material>
+     <mu1 value="0.001"/>
+     <mu2 value="0.001"/>
+   </gazebo>
 </robot>
