Commit message: cleaned workspace

File: src/my_robot_description/urdf/mobile_base.ros2_control.xacro (robot description, xacro)
@@ -1,23 +1,23 @@
 <?xml version="1.0"?>
 <robot xmlns:xacro="http://www.ros.org/wiki/xacro">
-  <ros2_control name="MobileBase" type="system">
-    <hardware>
-    <!-- <plugin>mock_components/GenericSystem</plugin>
-     <param name="calculate_dynamics">true</param>
-    -->
-    <plugin>
-      mobile_base_hardware/MobileBaseHardwareInterface
-    </plugin>
-    </hardware>
-    <joint name="base_right_wheel_joint">
-        <command_interface name="velocity"/>
-        <state_interface name="position"/>
-        <state_interface name="velocity"/>
-    </joint>
-      <joint name="base_left_wheel_joint">
-        <command_interface name="velocity"/>
-        <state_interface name="position"/>
-        <state_interface name="velocity"/>
-    </joint>
-  </ros2_control>
- </robot>
+    <ros2_control name="MobileBase" type="system">
+        <hardware>
+            <!-- <plugin>mock_components/GenericSystem</plugin>
+            <param name="calculate_dynamics">true</param> -->
+            <plugin>mobile_base_hardware/MobileBaseHardwareInterface</plugin>
+            <param name="left_motor_id">10</param>
+            <param name="right_motor_id">20</param>
+            <!-- <param name="dynamixel_port">/dev/ttyUSB0</param> -->
+        </hardware>
+        <joint name="base_right_wheel_joint">
+            <command_interface name="velocity" />
+            <state_interface name="position" />
+            <state_interface name="velocity" />
+        </joint>
+        <joint name="base_left_wheel_joint">
+            <command_interface name="velocity" />
+            <state_interface name="position" />
+            <state_interface name="velocity" />
+        </joint>
+    </ros2_control>
+</robot>

File: src/my_robot_description/urdf/mobile_base.xacro (robot description, xacro)
@@ -27,6 +27,6 @@
         </link>
     </xacro:macro>
-    <xacro:wheel_link prefix="right"/>
-    <xacro:wheel_link prefix="left"/>
+    <xacro:wheel_link prefix="right" />
+    <xacro:wheel_link prefix="left" />
     <link name="caster_wheel_link">
         <visual>

File: src/my_robot_description/urdf/my_robot.urdf.xacro (robot description, xacro)
@@ -3,4 +3,4 @@
     <xacro:include filename="common_properties.xacro" />
     <xacro:include filename="mobile_base.xacro" />
-    <xacro:include filename="mobile_base.ros2_control.xacro"/>
+    <xacro:include filename="mobile_base.ros2_control.xacro" />
 </robot>
