Commit message: integrated_lidar_and_motordriver

File: src/my_robot_description/urdf/common_properties.xacro (robot description, xacro)
@@ -7,3 +7,12 @@
         <color rgba="0.5 0.5 0.5 1" />
     </material>
+    <material name="yellow">
+        <color rgba="1.0 1.0 0 1" />
+    </material>
+    <material name="orange">
+        <color rgba="1.0 0.5 0 1" />
+    </material>
+    <material name="black">
+        <color rgba="0 0 0 1" />
+    </material>
 </robot>

File: src/my_robot_description/urdf/my_robot.urdf.xacro (robot description, xacro)
@@ -4,3 +4,14 @@
     <xacro:include filename="mobile_base.xacro" />
     <xacro:include filename="mobile_base.ros2_control.xacro" />
+    <!-- <xacro:include filename="arm.xacro"/>
+    <xacro:include filename="arm.ros2_control.xacro"/> -->
+    <xacro:include filename="lidar.xacro"/>
+    <!-- <xacro:include filename="lidar.ros2_control.xacro"/> -->
+    <!-- <xacro:lidar/> -->
+    <!-- <xacro:lidar/> -->
+    <!-- <joint name="mobile_base_arm_joint" type="fixed">
+        <parent link="base_link" />
+        <child link="arm_base_link" />
+        <origin xyz="${base_length / 4.0} 0 ${base_height}" rpy="0 0 0" />
+    </joint> -->
 </robot>
