Commit message: updated robot description,improving driver code

File: src/my_robot_description/urdf/lidar.xacro (robot description, xacro)
@@ -2,11 +2,30 @@
 <robot xmlns:xacro="http://www.ros.org/wiki/xacro" name="lidar_model">
  <xacro:property name="_10cm" value="0.1" />
- <xacro:property name="lidar_length" value="0.2" />
- <xacro:property name="lidar_radius" value="0.1"/>
+ <xacro:property name="lidar_length" value="0.06" />
+ <xacro:property name="lidar_radius" value="0.04"/>
+ <xacro:property name="battery_length" value="0.11" />
+ <xacro:property name="battery_width" value="0.09" />
+ <xacro:property name="battery_height" value="0.065" />
+  <!--battery joint-->
+  <joint name="battery_joint" type="fixed">
+    <parent link="base_link"/>
+    <child link="battery_link"/>
+    <origin xyz="${base_length/5.0+0.025} 0 ${base_height}" rpy="0 0 0"/>
+  </joint>
+  <!-- battery link -->
+   <link name="battery_link">
+        <visual>
+            <geometry>
+                <box size="${battery_length} ${battery_width} ${battery_height}" />
+            </geometry>
+            <origin xyz="0 0 ${base_height/2.0}" rpy="0 0 0" />
+            <material name="yellow" />
+        </visual>
+    </link>
    <!-- Lidar Joint -->
   <joint name="lidar_joint" type="fixed">
-    <parent link="base_link"/>
+    <parent link="battery_link"/>
     <child link="lidar_link"/>
-    <origin xyz="0.15 0 0.2" rpy="0 0 0"/>
+    <origin xyz="0 0 ${battery_height+0.04}" rpy="0 0 0"/>
   </joint>
   <!-- Lidar Link -->
@@ -16,5 +35,5 @@
         <cylinder length="${lidar_length}" radius="${lidar_radius}"/>
       </geometry>
-      <origin xyz="0 0 0.01" rpy="0 0 0"/>
+      <origin xyz="0 0 0.0" rpy="0 0 0"/>
       <material name="black"/>
     </visual>

File: src/my_robot_description/urdf/mobile_base.xacro (robot description, xacro)
@@ -1,9 +1,9 @@
 <?xml version="1.0"?>
 <robot xmlns:xacro="http://www.ros.org/wiki/xacro">
-    <xacro:property name="base_length" value="0.6" />
-    <xacro:property name="base_width" value="0.4" />
-    <xacro:property name="base_height" value="0.2" />
-    <xacro:property name="wheel_radius" value="0.1" />
-    <xacro:property name="wheel_length" value="0.05" />
+    <xacro:property name="base_length" value="0.35" />
+    <xacro:property name="base_width" value="0.15" />
+    <xacro:property name="base_height" value="0.07" />
+    <xacro:property name="wheel_radius" value="0.033" />
+    <xacro:property name="wheel_length" value="0.04" />
     <link name="base_footprint" />
     <link name="base_link">
@@ -13,5 +13,5 @@
             </geometry>
             <origin xyz="0 0 ${base_height / 2.0}" rpy="0 0 0" />
-            <material name="blue" />
+            <material name="grey" />
         </visual>
     </link>
@@ -23,5 +23,5 @@
                 </geometry>
                 <origin xyz="0 0 0" rpy="${pi / 2.0} 0 0" />
-                <material name="grey" />
+                <material name="black" />
             </visual>
         </link>
@@ -35,5 +35,5 @@
             </geometry>
             <origin xyz="0 0 0" rpy="0 0 0" />
-            <material name="grey" />
+            <material name="black"/>
         </visual>
     </link>
